File: Hardware/rev2/SAML10_DEV_2.brd (EAGLE design)
At the start: 38.1 x 25.4 mm, 20 parts, among them J1 CORTEX_DEBUG_PTH, Y1 32.768kHz

Commit message: final rev2 files
move to prototype production
Parts:
- moved D2 16.0 mm to (12.6, 19.5)
- moved R2 15.8 mm to (15.8, 19.4)
- moved JP1 13.5 mm to (16.7, 17.9), turned to 90 degrees
- moved R3 7.37 mm to (6.86, 11.7), turned to 270 degrees
- moved S1 7.37 mm to (5.40, 18.6), turned to 0 degrees
- moved C3 4.28 mm to (12.5, 17.1)
- moved C10 1.17 mm to (30.4, 6.72)
- moved C9 0.76 mm to (27.6, 8.67)
- moved U1 0.39 mm to (21.1, 8.85)
- turned J1 to 90 degrees
Connections:
- removed net VDDAN: J3.2
- net RESET: no longer J2.11
- net SWCLK: no longer J2.13
- net SWDIO: no longer J2.14
- net VIN: no longer J3.14
Routing:
- net VCC: track 0.00 -> 41.1 mm, vias 0 -> 3
- net SWCLK: track 0.00 -> 26.3 mm, vias 0 -> 1
- net RESET: track 0.00 -> 25.8 mm
- net PTC_X: track 0.00 -> 20.4 mm
- net SWDIO: track 0.00 -> 19.4 mm, vias 0 -> 1
- net PTC_Y: track 0.00 -> 18.7 mm
- net GPIO9: track 0.00 -> 17.0 mm
- net GPIO0: track 0.00 -> 16.5 mm
- net SCL: track 0.00 -> 16.1 mm
- net SDA: track 0.00 -> 14.0 mm
- net GPIO16: track 0.00 -> 13.9 mm
- net GPIO8: track 0.00 -> 13.6 mm
- net GPIO1: track 0.00 -> 13.2 mm
- net GPIO15: track 0.00 -> 12.6 mm
- net GPIO10: track 0.00 -> 12.2 mm
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Other:
- board text added: "VOUT LED"
- board text removed: "Check VCC connections:"
- board text removed: "RESET"
- board text removed: "VCC to VDDCORE, VDDANA,VDDIO GNDANA to GND"
- board text removed: "VIN"

Commit message: Swapped RESET pull up
from 4.7K to 10K
Parts:
- R3: value 4.7k -> 10k
Changed lines of the file:
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@@
 <?xml version="1.0" encoding="utf-8"?>
 <!DOCTYPE eagle SYSTEM "eagle.dtd">
-<eagle version="9.5.2">
+<eagle version="9.6.2">
 <drawing>
 <settings>
@@
 <layer number="115" name="ReferenceISLANDS" color="7" fill="1" visible="no" active="yes"/>
 <layer number="116" name="Patch_BOT" color="9" fill="4" visible="yes" active="yes"/>
+<layer number="117" name="PM_Ref" color="7" fill="1" visible="no" active="no"/>
 <layer number="118" name="Rect_Pads" color="7" fill="1" visible="no" active="yes"/>
+<layer number="119" name="PF_Ref" color="7" fill="1" visible="no" active="no"/>
+<layer number="120" name="WFL_Ref" color="7" fill="1" visible="no" active="no"/>
 <layer number="121" name="_tsilk" color="7" fill="1" visible="yes" active="yes"/>
 <layer number="122" name="_bsilk" color="7" fill="1" visible="yes" active="yes"/>
@@
 <attribute name="VALUE" x="12.5095" y="17.8435" size="0.6096" layer="27" font="vector" ratio="20" rot="R180" align="top-center"/>
 </element>
-<element name="R3" library="SparkFun-Resistors" library_urn="urn:adsk.eagle:library:532" package="0603" package3d_urn="urn:adsk.eagle:package:39650/1" value="4.7k" x="6.858" y="11.684" smashed="yes" rot="R270">
+<element name="R3" library="SparkFun-Resistors" package="0603" value="10k" x="6.858" y="11.684" smashed="yes" rot="R270">
 <attribute name="NAME" x="7.62" y="11.684" size="0.6096" layer="25" font="vector" ratio="20" rot="R270" align="bottom-center"/>
-<attribute name="PROD_ID" value="RES-07857" x="6.858" y="11.684" size="1.778" layer="27" rot="R270" display="off"/>
-<attribute name="VALUE" x="6.096" y="11.684" size="0.6096" layer="27" font="vector" ratio="20" rot="R270" align="top-center"/>
+<attribute name="PROD_ID" value="RES-00824" x="6.858" y="11.684" size="1.778" layer="27" rot="R270" display="off"/>
+<attribute name="VALUE" value="10k" x="6.096" y="11.684" size="0.6096" layer="27" font="vector" ratio="20" rot="R270" align="top-center"/>
 </element>
 <element name="S1" library="SparkFun-Switches" library_urn="urn:adsk.eagle:library:535" package="TACTILE_SWITCH_SMD_4.6X2.8MM" package3d_urn="urn:adsk.eagle:package:40176/1" value="" x="5.3975" y="18.6055" smashed="yes">
